Commit message: improve: Update Docker build context and file paths for Stereo Vision Node and app data

File: stereo_vision/urdf/NuroMower.urdf (robot description, URDF)
Before this commit: robot worx_mower, 3 links, 2 joints
Links:
- removed link base_footprint
- added link gps_link; visual cylinder length=0.02 radius=0.05
- link base_link: geometry visual box size=0.6 0.4 0.3
- link camera_link: geometry visual box size=0.03 0.12 0.03
Joints:
- removed joint base_footprint_joint
- added joint gps_joint: type fixed, parent base_link, child gps_link, origin xyz={GPS_OFFSET_X} 0.0 {GPS_HEIGHT_Z} rpy=0.0 0.0 0.0
- joint camera_joint: origin xyz=0.20 0.0 0.15 rpy=0 0 0 -> xyz={CAMERA_OFFSET_X} 0.0 {CAMERA_HEIGHT_Z} rpy=0.0 {CAMERA_PITCH_Y} 0.0
